File: Hardware/Audio/AudioCoprocessor/AudioCoproccessor.sch (EAGLE design)
At the start: 22 parts, among them IC1 AD7524JN, IC2 74LS32N, IC3 74HC573N, IC4 7400N, IC5 74HC573N, IC6 74S74N, IC7 LM358N, J2 RCJ-014, U1 W65C02SP

Commit message: regrettably I don't remember what I changed since the last commit
Other:
- note added: "DAC selected when: A15 high PHI2 high RWB low"
- note added: "IRQ-generating counter"
- note added: "clock speed jumper"
- note added: "dual ported SRAM"
- note added: "op amp power pins"
- note added: "reconstruction filter"
- note added: "unused, left unconnected in case needed for bodge work"
- moved on the sheet: IC2D
Changed lines of the file:
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@@
 <plain>
 <text x="254" y="160.02" size="1.778" layer="97">or TLC7524</text>
-<text x="165.1" y="193.04" size="1.778" layer="95">DAC gets updated from latch when interrupt is triggered
+<text x="139.7" y="195.58" size="2.54" layer="95">DAC gets updated from latch when interrupt is triggered
 this gives the APU flexibility wrt when it updates the output</text>
+<text x="297.18" y="127" size="1.778" layer="97">op amp power pins</text>
+<text x="271.78" y="58.42" size="1.778" layer="97">unused, left unconnected in case needed for bodge work</text>
+<text x="322.58" y="203.2" size="2.54" layer="97">reconstruction filter</text>
+<text x="5.08" y="96.52" size="2.54" layer="97">dual ported SRAM</text>
+<text x="25.4" y="-38.1" size="2.54" layer="97">IRQ-generating counter</text>
+<text x="-78.74" y="10.16" size="2.54" layer="97">clock speed jumper</text>
+<text x="185.42" y="66.04" size="2.54" layer="97">DAC selected when:
+A15 high
+PHI2 high
+RWB low</text>
 </plain>
 <instances>
 <instance part="U1" gate="G$1" x="129.54" y="68.58" smashed="yes">
 <attribute name="PART" x="119.38" y="96.52" size="1.778" layer="95" rot="MR180"/>
-<attribute name="VALUE" x="119.38" y="27.94" size="1.778" layer="95"/>
+<attribute name="VALUE" x="119.38" y="27.94" size="2.54" layer="95"/>
 </instance>
 <instance part="MOTHERBOARD" gate="A" x="-116.84" y="124.46" smashed="yes" rot="R90">
@@
 <attribute name="VALUE" x="185.42" y="93.98" size="1.778" layer="96" rot="R90"/>
 </instance>
-<instance part="IC2" gate="D" x="2.54" y="200.66" smashed="yes" rot="R90">
-<attribute name="NAME" x="-3.175" y="193.04" size="1.778" layer="95" rot="R90"/>
-<attribute name="VALUE" x="10.16" y="193.04" size="1.778" layer="96" rot="R90"/>
+<instance part="IC2" gate="D" x="276.86" y="76.2" smashed="yes" rot="R90">
+<attribute name="NAME" x="271.145" y="68.58" size="1.778" layer="95" rot="R90"/>
+<attribute name="VALUE" x="284.48" y="66.04" size="1.778" layer="96" rot="R90"/>
 </instance>
 <instance part="GND5" gate="1" x="5.08" y="25.4" smashed="yes">
@@
 <wire x1="55.88" y1="-10.16" x2="58.42" y2="-10.16" width="0.1524" layer="91"/>
 <wire x1="58.42" y1="-10.16" x2="109.22" y2="-10.16" width="0.1524" layer="91"/>
-<wire x1="109.22" y1="-10.16" x2="215.9" y2="-10.16" width="0.1524" layer="91"/>
-<wire x1="215.9" y1="-10.16" x2="215.9" y2="190.5" width="0.1524" layer="91"/>
+<wire x1="109.22" y1="-10.16" x2="220.98" y2="-10.16" width="0.1524" layer="91"/>
+<wire x1="220.98" y1="-10.16" x2="220.98" y2="190.5" width="0.1524" layer="91"/>
 <pinref part="IC1" gate="G$1" pin="!WR"/>
-<wire x1="215.9" y1="190.5" x2="248.92" y2="190.5" width="0.1524" layer="91"/>
+<wire x1="220.98" y1="190.5" x2="248.92" y2="190.5" width="0.1524" layer="91"/>
 <pinref part="U1" gate="G$1" pin="IRQB"/>
 <wire x1="114.3" y1="38.1" x2="109.22" y2="38.1" width="0.1524" layer="91"/>
