File: Hardware/Cartridge/BasicRomCard8K.brd (EAGLE design)
At the start: 47.9 x 47.9 mm, 3 parts

Commit message: regrettably I don't remember what I changed since the last commit
Connections:
- net N$10 renamed A0
- net N$11 renamed A1
- net N$12 renamed A2
- net N$13 renamed A3
- net N$14 renamed A4
- net N$15 renamed A5
- net N$16 renamed A6
- net N$17 renamed A7
- net N$18 renamed A12
- net N$19 renamed A8
- net N$2 renamed D0
- net N$20 renamed A9
- net N$21 renamed A10
- net N$22 renamed A11
- net N$23 renamed !WE
- net N$24 renamed !OE
- net N$26 renamed !CS
- net N$3 renamed D1
- net N$4 renamed D2
- net N$5 renamed D3
- net N$6 renamed D4
- net N$7 renamed D5
- net N$8 renamed D6
- net N$9 renamed D7
- new net !IRQ: U$1.P$34
- new net !RESET: U$1.P$20
- new net A13: U$1.P$36
- new net A14: U$1.P$22
- new net CLK: U$1.P$18
- new net I2CC: U$1.P$5
- new net I2CD: U$1.P$4
- new net RDY: U$1.P$21
