File: Hardware/VideoOut/vidgen_only_r3.brd (EAGLE design)
At the start: 138.4 x 100 mm, 78 parts, among them IC34 74HC164N, IC35 74LS151N, IC36 4040N, IC37 74AS30N, IC38 74LS74N, IC39 7400N, IC40 4040N, IC41 7400N, IC42 74LS74N, IC43 7400N, IC44 7486N, IC45 7400N, IC46 74S257N, IC47 74S257N, IC48 74HC563N, IC49 74LS08N, IC50 74LS08N, IC51 4040N, IC52 4040N, IC53 7404N, J1 RCJ-014, J2 TX24-40R-12ST-H1E

Commit message: regrettably I don't remember what I changed since the last commit
Parts:
- IC48: value 74HC563N -> 74HC564N
Connections:
- new net N$21: IC48.11, IC51.9
- net XCLK: no longer IC48.11
