File: Hardware/VideoOut/vidgen_only_r3.sch (EAGLE design)
At the start: 78 parts, among them IC34 74HC164N, IC35 74LS151N, IC36 4040N, IC37 74AS30N, IC38 74LS74N, IC39 7400N, IC40 4040N, IC41 7400N, IC42 74LS74N, IC43 7400N, IC44 7486N, IC45 7400N, IC46 74S257N, IC47 74S257N, IC48 74HC563N, IC49 74LS08N, IC50 74LS08N, IC51 4040N, IC52 4040N, IC53 7404N, J1 RCJ-014, J2 TX24-40R-12ST-H1E

Commit message: regrettably I don't remember what I changed since the last commit
Parts:
- IC48: value 74HC563N -> 74HC564N; device 74xx-us:74HC563N -> 74xx-us:74HC564N
Connections:
- new net N$21: IC48A.CLK, IC51A.Q1
- net XCLK: no longer IC48A.C
Changed lines of the file:
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@@
 <part name="GND32" library="supply1" library_urn="urn:adsk.eagle:library:371" deviceset="GND" device=""/>
 <part name="GND33" library="supply1" library_urn="urn:adsk.eagle:library:371" deviceset="GND" device=""/>
-<part name="IC48" library="74xx-us" library_urn="urn:adsk.eagle:library:88" deviceset="74*563" device="N" package3d_urn="urn:adsk.eagle:package:16429/2" technology="HC"/>
+<part name="IC48" library="74xx-us" library_urn="urn:adsk.eagle:library:88" deviceset="74*564" device="N" package3d_urn="urn:adsk.eagle:package:16429/2" technology="HC"/>
 <part name="GND37" library="supply1" library_urn="urn:adsk.eagle:library:371" deviceset="GND" device=""/>
 <part name="IC49" library="74xx-us" library_urn="urn:adsk.eagle:library:88" deviceset="74*08" device="N" package3d_urn="urn:adsk.eagle:package:16407/2" technology="LS"/>
@@
 <wire x1="27.94" y1="269.24" x2="-12.7" y2="269.24" width="0.1524" layer="91"/>
 <junction x="-12.7" y="269.24"/>
-<pinref part="IC48" gate="A" pin="C"/>
 <pinref part="IC51" gate="A" pin="P1"/>
-<wire x1="109.22" y1="414.02" x2="27.94" y2="414.02" width="0.1524" layer="91"/>
-<wire x1="27.94" y1="414.02" x2="27.94" y2="406.4" width="0.1524" layer="91"/>
 <wire x1="-12.7" y1="269.24" x2="-12.7" y2="406.4" width="0.1524" layer="91"/>
 <wire x1="-12.7" y1="406.4" x2="27.94" y2="406.4" width="0.1524" layer="91"/>
-<junction x="27.94" y="406.4"/>
 <label x="17.78" y="406.4" size="1.778" layer="95"/>
 <label x="-10.16" y="269.24" size="1.778" layer="95"/>
@@
 </segment>
 </net>
+<net name="N$21" class="0">
+<segment>
+<pinref part="IC51" gate="A" pin="Q1"/>
+<pinref part="IC48" gate="A" pin="CLK"/>
+<wire x1="53.34" y1="406.4" x2="60.96" y2="414.02" width="0.1524" layer="91"/>
+<wire x1="60.96" y1="414.02" x2="109.22" y2="414.02" width="0.1524" layer="91"/>
+</segment>
+</net>
