File: Hardware/Blitter/vdma_only_v2.sch (EAGLE design)
At the start: 82 parts, among them IC1 74S08N, IC10 74HC191N, IC11 74HC191N, IC12 74HC191N, IC13 74HC191N, IC14 74HC191N, IC15 74HC191N, IC16 74HC573N, IC17 74HC573N, IC18 7432N, IC19 74LS257N, IC2 74HC191N, IC20 7430N, IC21 7400N, IC22 74LS257N, IC23 74LS257N, IC24 74LS257N, IC25 74LS257N, IC26 74LS257N, IC27 74LS257N, IC28 74LS257N, IC29 74LS257N, IC3 74HC573N, IC30 74HC573N, IC31 7400N, IC32 7432N, IC4 74HC191N, IC5 74HC573N, IC53 7404N, IC54 74LS07N, IC6 74HC573N, IC7 74HC573N, IC8 74HC573N, IC9 74LS74N, J1 TX25-40P-6ST-H1E, J2 TX25-40P-6ST-H1E

Commit message: update blitter
Parts:
- added C41: (no value), rcl:C-US025-024X044
- added IC33: 7400N, 74xx-us:7400N
Connections:
- removed net !DMAIRQEN: IC32A.I1, IC53B.O
- removed net N$100: IC32A.I0, IC9B.!Q
- removed net N$213: IC20A.O, IC53D.I
- removed net N$214: IC31C.I0, IC53D.O
- new net N$47: IC1A.O, IC33B.I1, IC33D.I0, IC33D.I1
- new net N$48: IC33C.I0, IC33D.O
- new net N$49: IC33A.I0, IC33A.I1, IC33B.O
- new net N$58: IC21D.I0, IC9B.Q
- new net N$66: IC20A.O, IC32A.I0
- new net XCLK: IC10A.CLK, IC12A.CLK, IC14A.CLK, IC2A.CLK, IC33A.O
- net !DMACLK!/!IDLE!: now also IC1C.I1; no longer IC31A.I1
- net !DMAIRQ: now also IC21D.O; no longer IC32A.O
- net !XRELOAD: now also IC33C.O; no longer IC1A.O
- net DMACLK/!IDLE!: now also IC33B.I0, IC33C.I1; no longer IC10A.CLK, IC12A.CLK, IC14A.CLK, IC2A.CLK
- net DMAIRQEN: now also IC21D.I1; no longer IC53B.I
- net GND: now also C41.2, IC31C.I0, IC31C.I1, IC53B.I, IC53D.I
- net N$16: now also IC31A.I0, IC32A.O; no longer IC1C.I1, IC31C.O
- net N$39: now also IC31A.I1; no longer IC31A.I0
- net TRANSEN: now also IC32A.I1; no longer IC31C.I1
- net VCC: now also C41.1
Other:
- note added: "When TRANSEN is low, an FF byte inhibits the VRAM write cycle"
- note removed: "When TRANSEN is high, an FF byte inhibits the VRAM write cycle"
- moved on the sheet: IC1C, IC31A, IC31C, IC32A, IC53B, IC53D

Commit message: regrettably I don't remember what I changed since the last commit
Parts:
- removed IC10, IC11, IC12, IC13, IC14, IC15, IC2, IC4: 74HC191N, 74xx-us:74HC191N
- removed IC19, IC22, IC23, IC24, IC25, IC26, IC27, IC28, IC29: 74LS257N, 74xx-us:74LS257N
- removed IC33: 7400N, 74xx-us:7400N
- added BANKMUX, GMUX0, GMUX1, GMUX2, GMUX3, VMUX0, VMUX1, VMUX2, VMUX3: 74LS257N, 74xx-us:74LS257N
- added GXFLIPPER, GYFLIPPER: 74AHC8541, 0_gametankparts:74AHC8541
- added GXH, GXL, GYH, GYL, VXH, VXL, VYH, VYL: 74HC163, 0_gametankparts:74HC163
- added PAD1, PAD2: (no value), wirepad:2,54/0,9
- renumbered IC16 to REG.VX, IC17 to REG.VY, IC3 to REG.FLAGS, IC30 to REG.COLOR, IC5 to REG.GX, IC6 to REG.GY, IC7 to REG.W, IC8 to REG.H, U$2 to CTR.W, U$3 to CTR.H
Connections:
- removed net N$107: IC12A.RCO, IC13A.CLK
- removed net N$109: IC14A.RCO, IC15A.CLK
- removed net XCLK: IC10A.CLK, IC12A.CLK, IC14A.CLK, IC2A.CLK, IC33A.O
- new net GX-CARRY: GXHG$1.ENT, GXLG$1.RCO
- new net GY-CARRY: GYHG$1.ENT, GYLG$1.RCO
- new net N$68: GXFLIPPERG$2.D5, GXHG$1.Q1
- new net N$72: GXFLIPPERG$2.D6, GXHG$1.Q2
- new net N$73: GYFLIPPERG$2.D0, GYLG$1.Q0
- new net N$74: GYFLIPPERG$2.D1, GYLG$1.Q1
- new net N$75: GYFLIPPERG$2.D2, GYLG$1.Q2
- new net N$76: GYFLIPPERG$2.D3, GYLG$1.Q3
- new net N$77: GYFLIPPERG$2.D4, GYHG$1.Q0
- new net N$78: GYFLIPPERG$2.D5, GYHG$1.Q1
- new net N$79: GYFLIPPERG$2.D6, GYHG$1.Q2
- new net N$80: GYFLIPPERG$2.T/!C, IC53B.O
- new net N$81: GXFLIPPERG$2.T/!C, IC31C.O
- new net ROWCOMPLETE: GYLG$1.ENT, IC53D.O, VYLG$1.ENT
- new net VX-CARRY: VXHG$1.ENT, VXLG$1.RCO
- new net VY-CARRY: VYHG$1.ENT, VYLG$1.RCO
- net !DMA-ENABLED: no longer IC12A.CTE, IC2A.CTE
- net !DMAMODE: now also GMUX0A.!A!/B, GMUX1A.!A!/B, GMUX2A.!A!/B, GMUX3A.!A!/B, VMUX0A.!A!/B, VMUX1A.!A!/B, VMUX2A.!A!/B, VMUX3A.!A!/B; no longer IC22A.!A!/B, IC23A.!A!/B, IC24A.!A!/B, IC25A.!A!/B, IC26A.!A!/B, IC27A.!A!/B, IC28A.!A!/B, IC29A.!A!/B
- net !DMASTART: now also GYHG$1._LOAD, GYLG$1._LOAD, VYHG$1._LOAD, VYLG$1._LOAD; no longer IC10A.LD, IC11A.LD, IC14A.LD, IC15A.LD
- net !ROWCOMPLETE: now also IC53D.I; no longer IC10A.CTE, IC14A.CTE
- net !VOE: now also VMUX3A.4Y; no longer IC25A.4Y
- net !VWE: now also VMUX1A.4Y; no longer IC23A.4Y
- net !XRELOAD: now also GXHG$1._LOAD, GXLG$1._LOAD, IC1A.O, VXHG$1._LOAD, VXLG$1._LOAD; no longer IC12A.LD, IC13A.LD, IC2A.LD, IC33C.O, IC4A.LD
- net A0: now also GMUX0A.1B, VMUX0A.1B; no longer IC22A.1B, IC26A.1B
- net A1: now also GMUX0A.2B, VMUX0A.2B; no longer IC22A.2B, IC26A.2B
- net A10: now also GMUX2A.4B, VMUX2A.4B; no longer IC24A.4B, IC28A.4B
- net A11: now also GMUX3A.1B, VMUX3A.1B; no longer IC25A.1B, IC29A.1B
- net A12: now also GMUX3A.2B, VMUX3A.2B; no longer IC25A.2B, IC29A.2B
- net A13: now also GMUX3A.3B, VMUX3A.3B; no longer IC25A.3B, IC29A.3B
- net A2: now also GMUX0A.3B, VMUX0A.3B; no longer IC22A.3B, IC26A.3B
- net A3: now also GMUX0A.4B, VMUX0A.4B; no longer IC22A.4B, IC26A.4B
- net A4: now also GMUX1A.1B, VMUX1A.1B; no longer IC23A.1B, IC27A.1B
- net A5: now also GMUX1A.2B, VMUX1A.2B; no longer IC23A.2B, IC27A.2B
- net A6: now also GMUX1A.3B, VMUX1A.3B; no longer IC23A.3B, IC27A.3B
- net A7: now also GMUX2A.1B, VMUX2A.1B; no longer IC24A.1B, IC28A.1B
- net A8: now also GMUX2A.2B, VMUX2A.2B; no longer IC24A.2B, IC28A.2B
- net A9: now also GMUX2A.3B, VMUX2A.3B; no longer IC24A.3B, IC28A.3B
- net COLORFILL: now also GMUX3A.4A; no longer IC29A.4A
- net DMA-ENABLED: now also GXHG$1.ENP, GXLG$1.ENP, GYHG$1.ENP, GYLG$1.ENP, VXHG$1.ENP, VXLG$1.ENP, VYHG$1.ENP, VYLG$1.ENP; no longer IC1D.I1
- net DMACLK/!IDLE!: now also GXHG$1.CLK, GXLG$1.CLK, GYHG$1.CLK, GYLG$1.CLK, VXHG$1.CLK, VXLG$1.CLK, VYHG$1.CLK, VYLG$1.CLK; no longer IC33B.I0, IC33C.I1
- net GND: now also BANKMUXA.G, GMUX0A.G, GMUX1A.G, GMUX2A.G, GMUX3A.G, GXFLIPPERG$2.!OE, GYFLIPPERG$2.!OE, PAD1.P, PAD2.P, VMUX0A.G, VMUX1A.G, VMUX2A.G, VMUX3A.G; no longer IC11A.CTE, IC11A.D, IC12A.D/!U, IC13A.CTE, IC13A.D, IC13A.D/!U, IC14A.D/!U, IC15A.CTE, IC15A.D, IC15A.D/!U, IC19A.G, IC22A.G, IC23A.G, IC24A.G, IC25A.G, IC26A.G, IC27A.G, IC28A.G, IC29A.G, IC31C.I0, IC31C.I1, IC4A.CTE, IC4A.D, IC53B.I, IC53D.I
- net N$1: now also GMUX0A.1Y; no longer IC26A.1Y
- net N$10: now also GMUX2A.3Y; no longer IC28A.3Y
- net N$11: now also GMUX2A.4Y; no longer IC28A.4Y
- net N$113: now also VYLG$1.P0; no longer IC14A.A
- net N$114: now also VYLG$1.P1; no longer IC14A.B
- net N$115: now also VYLG$1.P2; no longer IC14A.C
- net N$116: now also VYLG$1.P3; no longer IC14A.D
- net N$117: now also VXHG$1.P0; no longer IC13A.A
- net N$118: now also VXHG$1.P1; no longer IC13A.B
- net N$119: now also VXHG$1.P2; no longer IC13A.C
- net N$12: now also GMUX3A.1Y; no longer IC29A.1Y
- net N$121: now also VXLG$1.P0; no longer IC12A.A
- net N$122: now also VXLG$1.P1; no longer IC12A.B
- net N$123: now also VXLG$1.P2; no longer IC12A.C
- net N$124: now also VXLG$1.P3; no longer IC12A.D
- net N$13: now also GMUX3A.2Y; no longer IC29A.2Y
- net N$14: now also GMUX3A.3Y; no longer IC29A.3Y
- net N$15: now also VMUX1A.4A; no longer IC23A.4A
- net N$160: now also VMUX0A.2A, VXLG$1.Q1; no longer IC12A.QB, IC22A.2A
- net N$161: now also VMUX0A.3A, VXLG$1.Q2; no longer IC12A.QC, IC22A.3A
- net N$162: now also VMUX0A.4A, VXLG$1.Q3; no longer IC12A.QD, IC22A.4A
- net N$163: now also VMUX1A.1A, VXHG$1.Q0; no longer IC13A.QA, IC23A.1A
- net N$164: now also VMUX1A.2A, VXHG$1.Q1; no longer IC13A.QB, IC23A.2A
- net N$165: now also VMUX1A.3A, VXHG$1.Q2; no longer IC13A.QC, IC23A.3A
- net N$167: now also VMUX2A.2A, VYLG$1.Q1; no longer IC14A.QB, IC24A.2A
- net N$168: now also VMUX2A.3A, VYLG$1.Q2; no longer IC14A.QC, IC24A.3A
- net N$169: now also VMUX2A.4A, VYLG$1.Q3; no longer IC14A.QD, IC24A.4A
- net N$17: now also GMUX1A.4Y; no longer IC27A.4Y
- net N$170: now also VMUX3A.1A, VYHG$1.Q0; no longer IC15A.QA, IC25A.1A
- net N$171: now also VMUX3A.2A, VYHG$1.Q1; no longer IC15A.QB, IC25A.2A
- net N$172: now also VMUX3A.3A, VYHG$1.Q2; no longer IC15A.QC, IC25A.3A
- net N$173: now also GMUX0A.1A, GXFLIPPERG$2.Y0; no longer IC26A.1A, IC2A.QA
- net N$174: now also GMUX0A.2A, GXFLIPPERG$2.Y1; no longer IC26A.2A, IC2A.QB
- net N$175: now also GMUX0A.3A, GXFLIPPERG$2.Y2; no longer IC26A.3A, IC2A.QC
- net N$176: now also GMUX0A.4A, GXFLIPPERG$2.Y3; no longer IC26A.4A, IC2A.QD
- net N$177: now also GMUX1A.1A, GXFLIPPERG$2.Y4; no longer IC27A.1A, IC4A.QA
- net N$178: now also GMUX1A.2A, GXFLIPPERG$2.Y5; no longer IC27A.2A, IC4A.QB
- net N$179: now also GMUX1A.3A, GXFLIPPERG$2.Y6; no longer IC27A.3A, IC4A.QC
- net N$18: now also GMUX3A.4Y; no longer IC29A.4Y
- net N$180: now also GMUX2A.1A, GYFLIPPERG$2.Y0; no longer IC10A.QA, IC28A.1A
- net N$181: now also GMUX2A.2A, GYFLIPPERG$2.Y1; no longer IC10A.QB, IC28A.2A
- net N$182: now also GMUX2A.3A, GYFLIPPERG$2.Y2; no longer IC10A.QC, IC28A.3A
- net N$183: now also GMUX2A.4A, GYFLIPPERG$2.Y3; no longer IC10A.QD, IC28A.4A
- net N$184: now also GMUX3A.1A, GYFLIPPERG$2.Y4; no longer IC11A.QA, IC29A.1A
- net N$185: now also GMUX3A.2A, GYFLIPPERG$2.Y5; no longer IC11A.QB, IC29A.2A
- net N$186: now also GMUX3A.3A, GYFLIPPERG$2.Y6; no longer IC11A.QC, IC29A.3A
- net N$19: now also GYLG$1.P0; no longer IC10A.A
- net N$2: now also GMUX0A.2Y; no longer IC26A.2Y
- net N$20: now also GYLG$1.P1; no longer IC10A.B
- net N$21: now also GYLG$1.P2; no longer IC10A.C
- net N$22: now also GYLG$1.P3; no longer IC10A.D
- net N$23: now also GXHG$1.P0; no longer IC4A.A
- net N$24: now also GXHG$1.P1; no longer IC4A.B
- net N$25: now also GXHG$1.P2; no longer IC4A.C
- net N$26: now also GYHG$1.P0; no longer IC11A.A
- net N$27: now also GXLG$1.P0; no longer IC2A.A
- net N$28: now also GXLG$1.P1; no longer IC2A.B
- net N$29: now also GXLG$1.P2; no longer IC2A.C
- net N$3: now also GMUX0A.3Y; no longer IC26A.3Y
- net N$30: now also GXLG$1.P3; no longer IC2A.D
- net N$31: now also GYHG$1.P1; no longer IC11A.B
- net N$32: now also GYHG$1.P2; no longer IC11A.C
- net N$35: now also VYHG$1.P0; no longer IC15A.A
- net N$36: now also VYHG$1.P1; no longer IC15A.B
- net N$37: now also VYHG$1.P2; no longer IC15A.C
- net N$4: now also GMUX0A.4Y; no longer IC26A.4Y
- net N$42: now also GXFLIPPERG$2.D3, GXLG$1.Q3; no longer IC2A.RCO, IC4A.CLK
- net N$43: now also GXFLIPPERG$2.D2, GXLG$1.Q2; no longer IC10A.RCO, IC11A.CLK
- net N$47: now also GXFLIPPERG$2.D1, GXLG$1.Q1; no longer IC1A.O, IC33B.I1, IC33D.I0, IC33D.I1
- net N$48: now also GXFLIPPERG$2.D0, GXLG$1.Q0; no longer IC33C.I0, IC33D.O
- net N$49: now also GXFLIPPERG$2.D4, GXHG$1.Q0; no longer IC33A.I0, IC33A.I1, IC33B.O
- net N$5: now also GMUX1A.1Y; no longer IC27A.1Y
- net N$50: now also BANKMUXA.1Y, VMUX1A.4B; no longer IC19A.1Y, IC23A.4B
- net N$6: now also GMUX1A.2Y; no longer IC27A.2Y
- net N$67: now also BANKMUXA.2Y, VMUX3A.4B; no longer IC19A.2Y, IC25A.4B
- net N$69: now also BANKMUXA.3Y, GMUX1A.4B; no longer IC19A.3Y, IC27A.4B
- net N$7: now also GMUX1A.3Y; no longer IC27A.3Y
- net N$70: now also BANKMUXA.4Y, GMUX3A.4B; no longer IC19A.4Y, IC29A.4B
- net N$8: now also GMUX2A.1Y; no longer IC28A.1Y
- net N$9: now also GMUX2A.2Y; no longer IC28A.2Y
- net OFFSCR_X: now also VXHG$1.Q3; no longer IC13A.QD
- net OFFSCR_Y: now also VYHG$1.Q3; no longer IC15A.QD
- net V/_G: now also BANKMUXA.!A!/B; no longer IC19A.!A!/B
- net VA0: now also VMUX0A.1Y; no longer IC22A.1Y
- net VA1: now also VMUX0A.2Y; no longer IC22A.2Y
- net VA10: now also VMUX2A.4Y; no longer IC24A.4Y
- net VA11: now also VMUX3A.1Y; no longer IC25A.1Y
- net VA12: now also VMUX3A.2Y; no longer IC25A.2Y
- net VA13: now also VMUX3A.3Y; no longer IC25A.3Y
- net VA2: now also VMUX0A.3Y; no longer IC22A.3Y
- net VA3: now also VMUX0A.4Y; no longer IC22A.4Y
- net VA4: now also VMUX1A.1Y; no longer IC23A.1Y
- net VA5: now also VMUX1A.2Y; no longer IC23A.2Y
- net VA6: now also VMUX1A.3Y; no longer IC23A.3Y
- net VA7: now also VMUX2A.1Y; no longer IC24A.1Y
- net VA8: now also VMUX2A.2Y; no longer IC24A.2Y
- net VA9: now also VMUX2A.3Y; no longer IC24A.3Y
- net VCC: now also BANKMUXA.1A, BANKMUXA.2A, BANKMUXA.3B, BANKMUXA.4B, GMUX1A.4A, GXHG$1._CLR, GXLG$1.ENT, GXLG$1._CLR, GYHG$1._CLR, GYLG$1._CLR, IC1D.I1, VMUX3A.4A, VXHG$1._CLR, VXLG$1.ENT, VXLG$1._CLR, VYHG$1._CLR, VYLG$1._CLR; no longer IC19A.1A, IC19A.2A, IC19A.3B, IC19A.4B, IC25A.4A, IC27A.4A
- net VG_OE: now also BANKMUXA.2B, BANKMUXA.4A; no longer IC19A.2B, IC19A.4A
- net VG_WE: now also BANKMUXA.1B, BANKMUXA.3A; no longer IC19A.1B, IC19A.3A
- net XDIR: now also IC31C.I0, IC31C.I1; no longer IC2A.D/!U, IC4A.D/!U
- net XODD: now also VMUX0A.1A, VXLG$1.Q0; no longer IC12A.QA, IC22A.1A
- net YDIR: now also IC53B.I; no longer IC10A.D/!U, IC11A.D/!U
- net YODD: now also VMUX2A.1A, VYLG$1.Q0; no longer IC14A.QA, IC24A.1A
Other:
- note added: "6ns"
- note added: "7ns"
- note added: "period 279.3 ns"
- moved on the sheet: IC18D, IC1C, IC20, IC21A, IC21B, IC21C, IC31A, IC31C, IC32A, IC53B, IC53D, J2

Commit message: Blitter V6 w/ 4-phase clock
Parts:
- added C42, C43, C44, C46: (no value), rcl:C-US025-024X044
- added CLK.SEQ: 74ALS08N, 74xx-us:74ALS08N
- added IC2: 74ALS04N, 74xx-us:74ALS04N
- added IC5: 74ALS00N, 74xx-us:74ALS00N
- added TRIGGER.INIT: 74LS74N, 74xx-us:74LS74N
Connections:
- net !DMAIRQ renamed !IRQ-OUT
- net DMAIRQEN renamed IRQ-ENABLE
- net N$58 renamed IRQ
- removed net !CLK28: IC1C.I0, IC53F.O
- removed net !DMA-ENABLED: CTR.WG$1.TE, IC32D.I1, IC9A.!Q
- removed net !DMACLK!/!IDLE!: CTR.HG$1.CP, CTR.WG$1.CP, IC1C.I1, IC53E.O
- removed net !DMASTART: CTR.HG$1.PL, CTR.WG$1.PL, GYHG$1._LOAD, GYLG$1._LOAD, IC1A.I0, IC31D.O, VYHG$1._LOAD, VYLG$1._LOAD
- removed net DMA-ENABLED: GXHG$1.ENP, GXLG$1.ENP, GYHG$1.ENP, GYLG$1.ENP, IC18C.I0, IC1B.I0, IC9A.Q, VXHG$1.ENP, VXLG$1.ENP, VYHG$1.ENP, VYLG$1.ENP
- removed net DMACLK/!IDLE!: GXHG$1.CLK, GXLG$1.CLK, GYHG$1.CLK, GYLG$1.CLK, IC1D.O, VXHG$1.CLK, VXLG$1.CLK, VYHG$1.CLK, VYLG$1.CLK
- removed net DMACLK/IDLE: IC32D.O, IC53E.I
- removed net DMASTART: IC31D.I0, IC31D.I1, IC9A.CLK, IC9B.CLK, U$5G$2.Y6
- new net !INIT: CTR.HG$1.PE, CTR.WG$1.PE, GYHG$1._LOAD, GYLG$1._LOAD, IC1A.I0, TRIGGER.INITA.CLR, TRIGGER.INITB.!Q, VYHG$1._LOAD, VYLG$1._LOAD
- new net !RUNNING: CTR.WG$1.TE, IC9A.!Q
- new net !TRIGGER: IC31D.O, TRIGGER.INITA.PRE
- new net N$58: IC31C.I1, TRIGGER.INITB.Q
- new net N$82: IC31C.O, IC9A.PRE, TRIGGER.INITB.CLR
- new net N$83: CLK.SEQD.I1, IC2C.O
- new net N$84: CLK.SEQD.I0, IC2D.O
- new net N$85: CLK.SEQB.I1, IC2A.O
- new net N$86: CLK.SEQC.I0, IC2B.O
- new net N$87: CTR.WG$1.PL, IC5A.O
- new net N$88: IC2E.O, IC9B.CLR
- new net P0: CLK.SEQD.O, CTR.WG$1.CP
- new net P1: CLK.SEQC.O, CTR.HG$1.CP, GXHG$1.CLK, GXLG$1.CLK, GYHG$1.CLK, GYLG$1.CLK, VXHG$1.CLK, VXLG$1.CLK, VYHG$1.CLK, VYLG$1.CLK
- new net P2: CLK.SEQB.O, IC31C.I0, IC5A.I0
- new net P3: CLK.SEQA.O, IC1C.I1, TRIGGER.INITB.CLK
- new net RUNNING: GXHG$1.ENP, GXLG$1.ENP, GYHG$1.ENP, GYLG$1.ENP, IC18C.I0, IC1B.I0, IC1C.I0, IC9A.Q, VXHG$1.ENP, VXLG$1.ENP, VYHG$1.ENP, VYLG$1.ENP
- new net TRIGGER-FLAG: TRIGGER.INITA.Q, TRIGGER.INITB.D
- new net TRIGGER-SELECT: IC2E.I, IC31D.I0, U$5G$2.Y6
- net !COPYDONE: no longer CTR.HG$1.PE
- net !ROWCOMPLETE: no longer CTR.WG$1.PE
- net CLK14: now also CLK.SEQA.I0, CLK.SEQB.I0, IC2B.I, IC2D.I; no longer IC1D.I0, IC32D.I0
- net CLK28: now also CLK.SEQA.I1, CLK.SEQC.I1, IC2A.I, IC2C.I; no longer IC53F.I
- net D0: now also IC31D.I1; no longer IC9A.D
- net D1: no longer IC9B.D
- net GND: now also C42.2, C43.2, C44.2, C46.2, IC9A.CLK, IC9A.D, IC9B.CLK, IC9B.D, TRIGGER.INITA.CLK, TRIGGER.INITA.D
- net N$81: now also IC53F.O; no longer IC31C.O
- net ROWCOMPLETE: now also IC5A.I1
- net VCC: now also C42.1, C43.1, C44.1, C46.1, CTR.HG$1.PL, TRIGGER.INITB.PRE; no longer IC1D.I1, IC9A.PRE, IC9B.CLR
- net XDIR: now also IC53F.I; no longer IC31C.I0, IC31C.I1
Other:
- note removed: "6ns"
- note removed: "period 279.3 ns"
- moved on the sheet: IC1B, IC21D, IC31C, IC31D, IC53C, IC53F, IC9A, IC9B, REG.COLOR

Commit message: Blitter fixes
Parts:
- added IC3: 74LS86N, 74xx-us:74LS86N
- added SJ1, SJ2, SJ3: (no value), jumper:SJ2W
Connections:
- removed net N$86: CLK.SEQC.I0, IC2B.O
- new net !SEQGEN_HIGH: CLK.SEQB.I1, CLK.SEQD.I0, IC3C.O
- new net !SEQGEN_LOW: CLK.SEQC.I1, CLK.SEQD.I1, IC3D.O
- new net N$89: IC3A.I0, IC3D.I1, SJ1.2
- new net P1LONG: CLK.SEQC.O, IC1D.I0
- new net SEQGEN_HIGH: CLK.SEQA.I1, CLK.SEQC.I0, IC3B.O
- new net SEQGEN_LOW: CLK.SEQA.I0, CLK.SEQB.I0, IC3A.O
- net CLK14: now also SJ2.3; no longer CLK.SEQA.I0, CLK.SEQB.I0, IC2B.I, IC2D.I
- net CLK28: now also IC53E.I; no longer CLK.SEQA.I1, CLK.SEQC.I1, IC2A.I, IC2C.I
- net CLK3_5: now also SJ1.1
- net CLK7: now also SJ1.3, SJ2.1
- net GND: now also IC3A.I1, IC3B.I1
- net N$83: now also IC3B.I0, IC3C.I1, SJ2.2; no longer CLK.SEQD.I1, IC2C.O
- net N$84: now also IC53E.O, SJ3.1; no longer CLK.SEQD.I0, IC2D.O
- net N$85: now also IC1D.I1, SJ3.2; no longer CLK.SEQB.I1, IC2A.O
- net P1: now also IC1D.O; no longer CLK.SEQC.O
- net VCC: now also IC3C.I0, IC3D.I0, SJ3.3
Other:
- moved on the sheet: CLK.SEQA, CLK.SEQB, CLK.SEQC, CLK.SEQD
