File: Hardware/Combined/cpu-blitter-inputs.sch (EAGLE design)
At the start: 149 parts, among them IC1 74S08N, IC12 74S08N, IC16 7404N, IC18 7432N, IC2 7404N, IC20 7430N, IC21 7400N, IC31 7400N, IC32 7432N, IC4 7404N, IC5 7400N, IC53 7404N, IC54 74LS07N, IC7 74S08N, IC9 74LS74N, J2 TX25-40P-6ST-H1E, U1 W65C02SP, U2 VIA

Commit message: Updates to combined board inc. new blitter features
Parts:
- removed G.RAM: SRAM_32K, 000_mychips2:SRAM_32K
- removed IC2: 7404N, 74xx-us:7404N
- removed SJ1, SJ2, SJ3: (no value), jumper:SJ2W
- removed U$1: SRAM_08K, 000_mychips2:SRAM_08K
- added IC3: 74HC573N, 74xx-us:74HC573N
- added U$4: AS6C4008, 0_gametankparts:AS6C4008
- added U$5: SRAM_32K, 0_gametankparts:SRAM_32K
Connections:
- net TRANSEN renamed !TRANSEN
- net VIDPAGE renamed VID_OUT_PAGE
- removed net !OE2: IC32C.I1
- removed net AUD_WAVE_N: AUDIOSLOT.8, WR_REG_DECODEG$2.Y5
- removed net GRAMBANK: G.RAMG$1.A14, REG.FLAGSA.4Q
- removed net N$34: IC1B.O, IC53C.I
- removed net P1LONG: CLK.SEQC.O, IC1D.I0
- new net !AUD_NMI: AUDIOSLOT.16
- new net !TILEMODE: IC1B.I1, IC1D.I1, REG.FLAGSA.5Q
- new net AUD_RESET: AUDIOSLOT.17
- new net AUD_SAMP_RATE_SEL: AUDIOSLOT.7
- new net GA14: GXFLIPPERG$2.Y7, U$4G$1.A14
- new net GA15: GYFLIPPERG$2.Y7, U$4G$1.A15
- new net GA16: IC3A.1Q, U$4G$1.A16
- new net GA17: IC3A.2Q, U$4G$1.A17
- new net GA18: IC3A.3Q, U$4G$1.A18
- new net GRAM_PAGE_SEL: IC3A.C, WR_REG_DECODEG$2.Y5
- new net GX-CARRY?: GXLG$1.RCO, IC1B.I0
- new net GY-CARRY?: GYLG$1.RCO, IC1D.I0
- new net N$150: GXHG$1.P3, REG.GXA.8Q
- new net N$151: GYHG$1.P3, REG.GYA.8Q
- new net N$84: REG.VYA.8Q, VYHG$1.P3
- new net RAM_PG_0: IC3A.7Q, U$5G$1.A13
- new net RAM_PG_1: IC3A.8Q, U$5G$1.A14
- net !CLK28: no longer SJ3.3
- net !RAMSEL: now also U$5G$1._CS; no longer U$1G$1._CE
- net !RE2: now also IC32C.I1, U$5G$1._OE; no longer U$1G$1._OE
- net !WE2: now also U$5G$1._WE; no longer U$1G$1._WE
- net !WRAP_X: now also IC3A.5Q; no longer REG.VXA.8Q
- net !WRAP_Y: now also IC3A.6Q; no longer REG.VYA.8Q
- net A0: now also U$5G$1.A0; no longer U$1G$1.A0
- net A1: now also U$5G$1.A1; no longer U$1G$1.A1
- net A10: now also U$5G$1.A10; no longer U$1G$1.A10
- net A11: now also U$5G$1.A11; no longer U$1G$1.A11
- net A12: now also U$5G$1.A12; no longer U$1G$1.A12
- net A2: now also U$5G$1.A2; no longer U$1G$1.A2
- net A3: now also U$5G$1.A3; no longer U$1G$1.A3
- net A4: now also U$5G$1.A4; no longer U$1G$1.A4
- net A5: now also U$5G$1.A5; no longer U$1G$1.A5
- net A6: now also U$5G$1.A6; no longer U$1G$1.A6
- net A7: now also U$5G$1.A7; no longer U$1G$1.A7
- net A8: now also U$5G$1.A8; no longer U$1G$1.A8
- net A9: now also U$5G$1.A9; no longer U$1G$1.A9
- net AUD_SQ1_N: no longer AUDIOSLOT.17
- net AUD_SQ1_X: no longer AUDIOSLOT.16
- net AUD_WAVE_X: no longer AUDIOSLOT.7
- net CLK14: no longer SJ2.3
- net CLK3_5: now also SEQGEN_XORA.I0, SEQGEN_XORD.I1; no longer SJ1.1
- net CLK7: now also SEQGEN_XORB.I0, SEQGEN_XORC.I1; no longer SJ1.3, SJ2.1
- net COLORFILL: now also IC5C.I1, REG.FLAGSA.4Q; no longer IC1B.I1, REG.GXA.8Q
- net D0: now also IC3A.1D, U$5G$1.D0; no longer U$1G$1.D0
- net D1: now also IC3A.2D, U$5G$1.D1; no longer U$1G$1.D1
- net D2: now also IC3A.3D, U$5G$1.D2; no longer U$1G$1.D2
- net D3: now also IC3A.4D, U$5G$1.D3; no longer U$1G$1.D3
- net D4: now also IC3A.5D, U$5G$1.D4; no longer U$1G$1.D4
- net D5: now also IC3A.6D, U$5G$1.D5; no longer U$1G$1.D5
- net D6: now also IC3A.7D, U$5G$1.D6; no longer U$1G$1.D6
- net D7: now also IC3A.8D, U$5G$1.D7; no longer U$1G$1.D7
- net DD0: now also U$4G$1.D0; no longer G.RAMG$1.D0
- net DD1: now also U$4G$1.D1; no longer G.RAMG$1.D1
- net DD2: now also U$4G$1.D2; no longer G.RAMG$1.D2
- net DD3: now also U$4G$1.D3; no longer G.RAMG$1.D3
- net DD4: now also U$4G$1.D4; no longer G.RAMG$1.D4
- net DD5: now also U$4G$1.D5; no longer G.RAMG$1.D5
- net DD6: now also U$4G$1.D6; no longer G.RAMG$1.D6
- net DD7: now also U$4G$1.D7; no longer G.RAMG$1.D7
- net GND: now also IC3A.OC, U$4G$1.!CE; no longer G.RAMG$1._CS
- net GX-CARRY: now also IC1B.O; no longer GXLG$1.RCO
- net GY-CARRY: now also IC1D.O; no longer GYLG$1.RCO
- net N$1: now also U$4G$1.A0; no longer G.RAMG$1.A0
- net N$10: now also U$4G$1.A9; no longer G.RAMG$1.A9
- net N$11: now also U$4G$1.A10; no longer G.RAMG$1.A10
- net N$12: now also U$4G$1.A11; no longer G.RAMG$1.A11
- net N$13: now also U$4G$1.A12; no longer G.RAMG$1.A12
- net N$14: now also U$4G$1.A13; no longer G.RAMG$1.A13
- net N$17: now also U$4G$1.!WE; no longer G.RAMG$1._WE
- net N$18: now also U$4G$1.!OE; no longer G.RAMG$1._OE
- net N$2: now also U$4G$1.A1; no longer G.RAMG$1.A1
- net N$3: now also U$4G$1.A2; no longer G.RAMG$1.A2
- net N$4: now also U$4G$1.A3; no longer G.RAMG$1.A3
- net N$41: now also IC5C.O; no longer IC53C.O
- net N$5: now also U$4G$1.A4; no longer G.RAMG$1.A4
- net N$6: now also U$4G$1.A5; no longer G.RAMG$1.A5
- net N$7: now also U$4G$1.A6; no longer G.RAMG$1.A6
- net N$8: now also U$4G$1.A7; no longer G.RAMG$1.A7
- net N$83: now also REG.VXA.8Q, VXHG$1.P3; no longer SEQGEN_XORB.I0, SEQGEN_XORC.I1, SJ2.2
- net N$85: now also GXFLIPPERG$2.D7, GXHG$1.Q3; no longer IC1D.I1, SJ3.2
- net N$88: now also IC5B.O; no longer IC2E.O
- net N$89: now also GYFLIPPERG$2.D7, GYHG$1.Q3; no longer SEQGEN_XORA.I0, SEQGEN_XORD.I1, SJ1.2
- net N$9: now also U$4G$1.A8; no longer G.RAMG$1.A8
- net P1: now also CLK.SEQC.O; no longer IC1D.O
- net RUNNING: now also IC5C.I0; no longer IC1B.I0
- net TRIGGER-SELECT: now also IC5B.I0, IC5B.I1; no longer IC2E.I
- net VCC: no longer SJ3.1, U$1G$1.CE2
- net VRAMBANK: now also IC3A.4Q; no longer REG.FLAGSA.5Q
Other:
- note added: "controlled by GX,GY highbit"
- note added: "controlled by register"
- moved on the sheet: IC1B, IC1D
