File: Hardware/Combined/signals.brd (EAGLE design)
At the start: 177.8 x 127 mm, 108 parts, among them IC2_AUD 74LS32N, IC36 4040N, IC37 74AS30N, IC39 7400N, IC40 4040N, IC41 7400N, IC43 7400N, IC44 7486N, IC45 7400N, IC46 74S257N, IC47 74S257N, IC48 74HC564N, IC4_AUD 7400N, IC53 7404N, IC6_AUD 74S74N, IC7_AUD LM358N, J2 TX24-40R-12ST-H1E, U1 W65C02SP

Commit message: Updates to combined board inc. new blitter features
Connections:
- removed net AUD_REG5: MOTHERBOARD.8
Changed lines of the file:
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@@
 <contactref element="MOTHERBOARD" pad="9"/>
-</signal>
-<signal name="AUD_REG5">
-<contactref element="MOTHERBOARD" pad="8"/>
 </signal>
 <signal name="AUD_REG6">
