File: Hardware/KiCad/LogicBoard/cpu-blitter-inputs.kicad_sch (KiCad schematic)
At the start: 0 parts

Commit message: mystery changes I forgot about on other computer and probably replicated and arent mergable oops
Other:
- added sheet Power (power.kicad_sch)
