File: Hardware/KiCad/avboard_tht2/avboard_tht2.kicad_pcb (KiCad board)
At the start: 4 copper layers, 177 x 152.1 mm, 139 parts, among them IC1 AS7C256C-15PCN, IC2_AUD0 74HC32, IC36 74HC4040, IC37 74HC30, IC39 74HC00, IC40 74HC4040, IC41 74HC00, IC43 74HC00, IC44 74HC86, IC45 74HC00, IC46 74HC257, IC47 74HC257, IC48 74HC564, IC4_AUD0 74HC00, IC53 74HC04, IC6_AUD0 74HC74, IC7_AUD0 LM358N, IC9 AS7C256C-15PCN, J1 5V, J2 5V, U1 W65C02S, U2 THS7374, U3 74VHC373, U4 74VHC373, U5 74VHC373, U8 74HC244, U9 74HC244

Commit message: fewer vias, simpler routing
Parts:
- AUDIO-DAC0: value TLC7524CDR -> TLC7524CN
- C14: value 680 pF -> 680pF
Routing:
- net MA4: track 149.9 -> 79.5 mm, vias 5 -> 3
- net /Composite Video Generator/PICTURE-ENABLE: track 148.6 -> 159.3 mm, vias 2 -> 0
- net VCC: track 57.4 -> 48.2 mm, vias 280 -> 297
- net /Audio Coprocessor/SysA7: track 53.8 -> 45.5 mm, vias 2 -> 1
- net VD1: track 60.8 -> 55.7 mm, vias 1 -> 0
- net VA2: track 72.2 -> 67.5 mm, vias 4 -> 2
- net /Audio Coprocessor/SysD1: track 40.3 -> 35.7 mm, vias 1 -> 2
- net Net-(IC4_AUD0D-O): track 79.2 -> 83.3 mm, vias 2 -> 1
- net /Composite Video Generator/LUM0: track 21.1 -> 17.4 mm
- net /Audio Coprocessor/DAC_SELECT: track 91.2 -> 88.0 mm, vias 2 -> 1
- net P3: track 52.6 -> 55.3 mm
- net P4: track 62.0 -> 64.6 mm, vias 4 -> 1
- net Net-(HBLANK_LATCH0A-D): track 38.5 -> 36.0 mm, vias 3 -> 2
- net Net-(IC53A-I): track 31.7 -> 29.8 mm
- net MA0: track 78.7 -> 76.8 mm, vias 9 -> 5
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