File: Hardware/KiCad/avboard_tht2/avboard_tht2.kicad_pcb (KiCad board)
At the start: 4 copper layers, 177 x 152.1 mm, 139 parts, among them IC1 AS7C256C-15PCN, IC2_AUD0 74HC32, IC36 74HC4040, IC37 74HC30, IC39 74HC00, IC40 74HC4040, IC41 74HC00, IC43 74HC00, IC44 74HC86, IC45 74HC00, IC46 74HC257, IC47 74HC257, IC48 74HC564, IC4_AUD0 74HC00, IC53 74HC04, IC6_AUD0 74HC74, IC7_AUD0 LM358N, IC9 AS7C256C-15PCN, J1 5V, J2 5V, U1 W65C02S, U2 THS7374, U3 74VHC373, U4 74VHC373, U5 74VHC373, U8 74HC244, U9 74HC244

Commit message: catchup commit for quote pkg stuff
Parts:
- moved C22 241.8 mm to (19.1, 41.9), turned to 0 degrees
- moved SCAN_DELAY0 202.0 mm to (92.7, 78.1), turned to 90 degrees
- moved C21 190.7 mm to (47.0, 56.5), turned to 0 degrees
- moved COL_CTR0 188.5 mm to (77.5, 66.7), turned to 90 degrees
- moved C15 175.2 mm to (47.6, 103.5), turned to 90 degrees
- moved C9 154.0 mm to (85.1, 98.4), turned to 90 degrees
- moved X_SCALER0 144.2 mm to (124.5, 66.7), turned to 90 degrees
- moved C40 143.3 mm to (73.7, 59.1), turned to -90 degrees
- moved C27 137.5 mm to (58.4, 98.4), turned to 90 degrees
- moved C8 129.3 mm to (124.5, 56.5)
- moved R15 128.9 mm to (77.5, 70.5), turned to 0 degrees
- moved C6 126.3 mm to (85.1, 70.5)
- moved IC40 124.9 mm to (29.2, 106.7), turned to 0 degrees
- moved C12 122.8 mm to (113.7, 94.0)
- moved C5 121.9 mm to (72.4, 70.5), turned to 180 degrees
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