File: Hardware/KiCad/avboard_tht2/signals_4.kicad_sch (KiCad schematic)
At the start: 22 parts, among them IC2_AUD0 74HC32, IC4_AUD0 74HC00, IC6_AUD0 74HC74, IC7_AUD0 LM358N, U1 W65C02S

Commit message: oops, forgot to add signals_4
Parts:
- AUDIO-DAC0: value TLC7524CDR -> TLC7524CN
Changed lines of the file:
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@@
 			)
 		)
-		(property "Value" "TLC7524CDR"
+		(property "Value" "TLC7524CN"
 			(at 396.24 60.96 0)
 			(show_name no)
