File: Hardware/KiCad/avboard_tht2/signals_4.kicad_sch (KiCad schematic)
At the start: 22 parts, among them IC2_AUD0 74HC32, IC4_AUD0 74HC00, IC6_AUD0 74HC74, IC7_AUD0 LM358N, U1 W65C02S

Commit message: catchup commit for quote pkg stuff
Connections:
- net SysD6: no longer J6.33
- net SysD7: now also J6.33
Changed lines of the file:
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@@
+		)
+	)
+	(label "SysD7"
+		(at 118.11 29.21 270)
+		(effects
+			(font
+				(size 1.27 1.27)
+			)
+			(justify right bottom)
 		)
 	)
@@
 		(effects
 			(font
-				(size 1.27 1.27)
-			)
-			(justify right bottom)
-		)
-	)
-	(label "SysD6"
-		(at 118.11 29.21 270)
-		(effects
-			(font
