File: Hardware/KiCad/LogicBoard_smt/Gamepad_ports.kicad_sch (KiCad schematic)
At the start: 11 parts

Commit message: catchup commit for quote pkg stuff
Parts:
- removed R6, R7: 3.3k, Resistor_SMD:R_0805_2012Metric, symbol cpu-blitter-inputs-eagle-import:R-US_0204/7
- added RN2, RN3: YC158TJR-0710KL, cpu-blitter-inputs:RESCAXE64P320X160X70-10N, symbol YC158TJR-0710KL:YC158TJR-0710KL
Connections:
- net VCC: now also RN2.10, RN2.5, RN3.10, RN3.5
- net at PAD1REG0.6 (5D), PORT1.1: now also RN2.9
- net at PAD1REG0.7 (6D), PORT1.2: now also RN2.8
- net at PAD1REG0.8 (7D), PORT1.3: now also RN2.7
- net at PAD1REG0.9 (8D), PORT1.4: now also RN2.6
- net at PAD1REG0.5 (4D), PORT1.6: now also RN2.1
- net at PAD1REG0.4 (3D), PORT1.9: now also RN2.2
- net at EXTRA_BUTTON_2.1, PAD2REG0.3 (2D): now also RN3.3
- net at PAD2REG0.4 (3D), PORT2.9: now also RN3.2
- net at PAD2REG0.5 (4D), PORT2.6: now also RN3.1
- net at PAD2REG0.6 (5D), PORT2.1: now also RN3.9
- net at PAD2REG0.7 (6D), PORT2.2: now also RN3.8
- net at PAD2REG0.8 (7D), PORT2.3: now also RN3.7
- net at PAD2REG0.9 (8D), PORT2.4: now also RN3.6
- net at EXTRA_BUTTON_1.1, PAD1REG0.3 (2D): now also RN2.3
