File: Hardware/KiCad/LogicBoard_smt/LogicBoard_smt.kicad_pcb (KiCad board)
At the start: 6 copper layers, 177.8 x 168.9 mm, 225 parts, among them IC1 7408N, IC12 7408N, IC16 MC74HC1GU04DFT1G, IC18 7432N, IC2 AP63205WU-7, IC20 7430N, IC21 7400N, IC3 74573N, IC31 7400N, IC32 7432N, IC4 7404N, IC5 7400N, IC53 7404N, IC7 7408N, IC9 7474N, J1 Conn_01x26_Socket, J2 JACK-PLUG0, J3 62684-502100ALF, J4 62684-502100ALF, U1 W65C02SP, U2 VIA, U3 GFXL, U4 GFXH, U5 GFYL, U6 GFYH, U7 74LVC2G07, U8 MCP130-xxxxTT, U9 TPS22919DCKR

Commit message: catchup commit for quote pkg stuff
Parts:
- removed R6, R7: 3.3k, Resistor_SMD:R_0805_2012Metric
- added RN2: YC158TJR-0710KL, cpu-blitter-inputs:RESCAXE64P320X160X70-10N, F.Cu at (94.1, 150.9)
- added RN3: YC158TJR-0710KL, cpu-blitter-inputs:RESCAXE64P320X160X70-10N, F.Cu at (147.4, 152.6)
Routing:
- net Net-(PAD1REG0A-7D): track 26.2 -> 46.2 mm, vias 0 -> 3
- net Net-(PAD1REG0A-8D): track 27.2 -> 45.2 mm, vias 0 -> 1
- net Net-(PAD2REG0A-5D): track 20.7 -> 37.1 mm, vias 0 -> 1
- net Net-(PAD1REG0A-6D): track 25.5 -> 41.3 mm, vias 0 -> 1
- net Net-(PAD1REG0A-5D): track 25.7 -> 38.7 mm, vias 0 -> 1
- net Net-(PAD2REG0A-4D): track 24.7 -> 35.6 mm
- net Net-(PAD2REG0A-7D): track 21.4 -> 31.7 mm, vias 0 -> 1
- net Net-(PAD2REG0A-8D): track 23.2 -> 32.1 mm, vias 0 -> 2
- net Net-(PAD2REG0A-3D): track 23.6 -> 31.5 mm
- net Net-(PAD2REG0A-6D): track 20.5 -> 26.5 mm, vias 0 -> 2
- net Net-(PAD1REG0A-3D): track 20.4 -> 25.8 mm, vias 1 -> 2
- net Net-(PAD2REG0A-2D): track 33.9 -> 37.3 mm, vias 1 -> 2
- net Net-(PAD1REG0A-4D): track 25.4 -> 27.6 mm, vias 1 -> 2
- net Net-(PAD1REG0A-2D): track 29.1 -> 31.3 mm
- net VCC: track 253.0 -> 254.6 mm, vias 126 -> 128
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Other:
- board text added: "GameTank CPU Board (SMT v. 4.6)"
- board text removed: "GameTank CPU Board (SMT v. 4.5)"
