File: Hardware/KiCad/ps_slash_2/ps2mkb/ps2mkb.kicad_sch (KiCad schematic)
At the start: 26 parts, among them SW1 SW_DIP_x08, U11 74HC32, U2 74HC573, U3 74HC688, U4 74HC573, U5 74HC03, U6 74HC04, U8 TS12A4515P, U9 74HC74

Commit message: catchup commit for quote pkg stuff
Other:
- note added: "Open collector NANDs"
Changed lines of the file:
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@@
+		)
+	)
+	(text "Open collector NANDs"
+		(exclude_from_sim no)
+		(at 376.936 113.792 0)
+		(effects
+			(font
+				(size 1.27 1.27)
+			)
 		)
 	)
